File: elrs-sim.kicad_sch (KiCad schematic)
At the start: 68 parts, among them IC1 SX1280IMLTRT, IC2 ESP8285, J1 Conn_01x04, J10 ESP_TX, J11 GND, J12 3.3V, J13 DP, J14 DN, J2 Conn_01x04, J3 Conn_01x04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

Commit message: Update main board
Parts:
- added C23: 1nF, Capacitor_SMD:C_0402_1005Metric, symbol Device:C
- C12: value 100nF -> 1uF
Connections:
- net at X3.3 (OUT): now also C23.2; no longer IC1.4 (XTA)
- new net: C23.1, IC1.4 (XTA)
Changed lines of the file:
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@@
 	(wire
 		(pts
+			(xy 200.66 229.87) (xy 200.66 233.68)
+		)
+		(stroke
+			(width 0)
+			(type default)
+		)
+	)
+	(wire
+		(pts
 			(xy 241.3 64.77) (xy 241.3 67.31)
 		)
@@
 	(wire
 		(pts
-			(xy 200.66 219.71) (xy 200.66 233.68)
+			(xy 200.66 219.71) (xy 200.66 222.25)
 		)
 		(stroke
@@
 		(dnp no)
 		(property "Reference" "X3"
-			(at 199.39 223.266 0)
+			(at 175.768 227.584 0)
 			(effects
 				(font
@@
 		)
 		(property "Value" "YSO510TP_52MHz"
-			(at 199.39 225.806 0)
+			(at 175.768 230.124 0)
 			(effects
 				(font
@@
 	)
 	(symbol
+		(lib_id "Device:C")
+		(at 200.66 226.06 0)
+		(unit 1)
+		(exclude_from_sim no)
+		(in_bom yes)
+		(on_board yes)
+		(dnp no)
+		(fields_autoplaced yes)
+		(property "Reference" "C23"
+			(at 204.47 224.7899 0)
+			(effects
+				(font
+					(size 1.27 1.27)
+				)
+				(justify left)
+			)
+		)
+		(property "Value" "1nF"
+			(at 204.47 227.3299 0)
+			(effects
+				(font
+					(size 1.27 1.27)
+				)
+				(justify left)
+			)
+		)
+		(property "Footprint" "Capacitor_SMD:C_0402_1005Metric"
+			(at 201.6252 229.87 0)
+			(effects
+				(font
+					(size 1.27 1.27)
+				)
+				(hide yes)
+			)
+		)
+		(property "Datasheet" "~"
+			(at 200.66 226.06 0)
+			(effects
+				(font
+					(size 1.27 1.27)
+				)
+				(hide yes)
+			)
+		)
+		(property "Description" "Unpolarized capacitor"
+			(at 200.66 226.06 0)
+			(effects
+				(font
+					(size 1.27 1.27)
+				)
+				(hide yes)
+			)
+		)
+		(property "LCSC" "C1523"
+			(at 204.47 224.7899 0)
+			(effects
+				(font
+					(size 1.27 1.27)
+				)
+				(hide yes)
+			)
+		)
+		(pin "1"
+		)
+		(pin "2"
+		)
+		(instances
+			(project "elrs-sim"
+				(path "/b1f5dd2a-859b-4a5a-8b1e-e98131c08e2f"
+					(reference "C23")
+					(unit 1)
+				)
+			)
+		)
+	)
+	(symbol
 		(lib_id "power:+3.3V")
 		(at 237.49 62.23 0)
@@
 			)
 		)
-		(property "Value" "100nF"
+		(property "Value" "1uF"
 			(at 104.14 187.9599 0)
 			(effects

Commit message: Update: Use SX1281, check BOM, hopefully final 0.0.1 prod files
Parts:
- IC1: value SX1280IMLTRT -> SX1281IMLTRT
Changed lines of the file:
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@@
 			)
 		)
-		(property "Value" "SX1280IMLTRT"
+		(property "Value" "SX1281IMLTRT"
 			(at 251.46 207.8543 0)
 			(effects
